File: Hardware/Grove_Monitor.sch (KiCad schematic (older format))
At the start: 23 parts, among them J3 QWIIC, J4 QWIIC, J5 Conn_01x03, J6 Conn_01x05, J7 Conn_01x03, J8 Conn_01x02, U1 PARTICLE_MESH

Commit message: V1.0 Complete
Parts:
- added J10, J9: Conn_01x01, Connectors:1X01, symbol Connector_Generic:Conn_01x01
- H1, H2, H3, H4: footprint MeowWolf_Hardware:STAND-OFF -> Openponics_Hardware:STAND-OFF_LARGE
- LOGO2: footprint Openponics_Logos:Openponics_Logo_Horizontal_10mm -> Openponics_Logos:Openponics_Logo_Horizontal_16mm
Connections:
- wire segments 164 -> 170
Changed lines of the file:
@@
 Title "Grove Monitoring System Adapter"
 Date "2019-02-16"
-Rev "00.04"
+Rev "V1.0"
 Comp "Openponics"
 Comment1 "Joel Bartlett"
@@
 F 0 "H1" H 10000 7100 45  0001 C CNN
 F 1 "STAND-OFF" H 10000 6900 45  0001 C CNN
-F 2 "MeowWolf_Hardware:STAND-OFF" H 10000 7150 20  0001 C CNN
+F 2 "Openponics_Hardware:STAND-OFF_LARGE" H 10000 7150 20  0001 C CNN
 F 3 "" H 10000 7000 50  0001 C CNN
 F 4 "XXX-00000" H 10078 7000 60  0001 L CNN "Field4"
@@
 F 0 "H2" H 10100 7100 45  0001 C CNN
 F 1 "STAND-OFF" H 10100 6900 45  0001 C CNN
-F 2 "MeowWolf_Hardware:STAND-OFF" H 10100 7150 20  0001 C CNN
+F 2 "Openponics_Hardware:STAND-OFF_LARGE" H 10100 7150 20  0001 C CNN
 F 3 "" H 10100 7000 50  0001 C CNN
 F 4 "XXX-00000" H 10178 7000 60  0001 L CNN "Field4"
@@
 F 0 "H3" H 10200 7100 45  0001 C CNN
 F 1 "STAND-OFF" H 10200 6900 45  0001 C CNN
-F 2 "MeowWolf_Hardware:STAND-OFF" H 10200 7150 20  0001 C CNN
+F 2 "Openponics_Hardware:STAND-OFF_LARGE" H 10200 7150 20  0001 C CNN
 F 3 "" H 10200 7000 50  0001 C CNN
 F 4 "XXX-00000" H 10278 7000 60  0001 L CNN "Field4"
@@
 F 0 "H4" H 10300 7100 45  0001 C CNN
 F 1 "STAND-OFF" H 10300 6900 45  0001 C CNN
-F 2 "MeowWolf_Hardware:STAND-OFF" H 10300 7150 20  0001 C CNN
+F 2 "Openponics_Hardware:STAND-OFF_LARGE" H 10300 7150 20  0001 C CNN
 F 3 "" H 10300 7000 50  0001 C CNN
 F 4 "XXX-00000" H 10378 7000 60  0001 L CNN "Field4"
@@
 A5
 Wire Wire Line
-	7150 3750 7050 3750
+	7150 3750 7100 3750
 $Comp
 L Connector_Generic:Conn_01x03 J7
@@
 A4
 Wire Wire Line
-	7150 4000 7050 4000
+	7150 4000 7100 4000
 Wire Wire Line
 	3400 7400 3450 7400
@@
 F 0 "LOGO2" H 8500 6818 60  0001 C CNN
 F 1 "OPENPONICS_LOGO" H 8500 7282 60  0001 C CNN
-F 2 "Openponics_Logos:Openponics_Logo_Horizontal_10mm" H 8500 7050 60  0001 C CNN
+F 2 "Openponics_Logos:Openponics_Logo_Horizontal_16mm" H 8500 7050 60  0001 C CNN
 F 3 "" H 8500 7050 60  0001 C CNN
 	1    8500 7050
@@
 	1    0    0    -1
 $EndComp
+$Comp
+L Connector_Generic:Conn_01x01 J9
+U 1 1 5C7A01C0
+P 7350 3600
+F 0 "J9" H 7430 3642 50  0000 L CNN
+F 1 "Conn_01x01" H 7430 3551 50  0000 L CNN
+F 2 "Connectors:1X01" H 7350 3600 50  0001 C CNN
+F 3 "~" H 7350 3600 50  0001 C CNN
+	1    7350 3600
+	1    0    0    -1
+$EndComp
+$Comp
+L Connector_Generic:Conn_01x01 J10
+U 1 1 5C7A01FC
+P 7350 3850
+F 0 "J10" H 7430 3892 50  0000 L CNN
+F 1 "Conn_01x01" H 7430 3801 50  0000 L CNN
+F 2 "Connectors:1X01" H 7350 3850 50  0001 C CNN
+F 3 "~" H 7350 3850 50  0001 C CNN
+	1    7350 3850
+	1    0    0    -1
+$EndComp
+Wire Wire Line
+	7150 3850 7100 3850
+Wire Wire Line
+	7100 3850 7100 4000
+Connection ~ 7100 4000
+Wire Wire Line
+	7100 4000 7050 4000
+Wire Wire Line
+	7150 3600 7100 3600
+Wire Wire Line
+	7100 3600 7100 3750
+Connection ~ 7100 3750
+Wire Wire Line
+	7100 3750 7050 3750
 $EndSCHEMATC
